File: SLMMK1/AR.sch (KiCad schematic (older format))
At the start: 32 parts, among them Q8 2N3904, SW1 SW_SPST, SW2 SW_SPST, SW3 SW_SPDT, U1 74HC14, U2 TL072

Commit message: Finished version
Parts:
- D1, D2, D3, D4, D5, D7, D8: footprint (none) -> Diodes_SMD:D_SOD-123F
- Q8: footprint Package_TO_SOT_THT:TO-92_Inline -> TO_SOT_Packages_THT:TO-92_Inline_Wide
Other:
- note added: "Attack Time\n"
- note added: "Release Time\n"
Changed lines of the file:
@@
 F 0 "D7" H 2600 2134 50  0000 C CNN
 F 1 "1N914" H 2600 2225 50  0000 C CNN
-F 2 "" H 2600 2350 50  0001 C CNN
+F 2 "Diodes_SMD:D_SOD-123F" H 2600 2350 50  0001 C CNN
 F 3 "~" H 2600 2350 50  0001 C CNN
 	1    2600 2350
@@
 F 0 "Q8" H 4091 2396 50  0000 L CNN
 F 1 "2N3904" H 4091 2305 50  0000 L CNN
-F 2 "Package_TO_SOT_THT:TO-92_Inline" H 4100 2275 50  0001 L CIN
+F 2 "TO_SOT_Packages_THT:TO-92_Inline_Wide" H 4100 2275 50  0001 L CIN
 F 3 "https://www.fairchildsemi.com/datasheets/2N/2N3904.pdf" H 3900 2350 50  0001 L CNN
 	1    3900 2350
@@
 F 0 "D8" H 3400 2966 50  0000 C CNN
 F 1 "1N5239B" H 3400 2875 50  0000 C CNN
-F 2 "" H 3400 2750 50  0001 C CNN
+F 2 "Diodes_SMD:D_SOD-123F" H 3400 2750 50  0001 C CNN
 F 3 "~" H 3400 2750 50  0001 C CNN
 	1    3400 2750
@@
 F 0 "D1" H 7050 1834 50  0000 C CNN
 F 1 "1N914" H 7050 1925 50  0000 C CNN
-F 2 "" H 7050 2050 50  0001 C CNN
+F 2 "Diodes_SMD:D_SOD-123F" H 7050 2050 50  0001 C CNN
 F 3 "~" H 7050 2050 50  0001 C CNN
 	1    7050 2050
@@
 F 0 "D2" H 7500 2266 50  0000 C CNN
 F 1 "1N914" H 7500 2175 50  0000 C CNN
-F 2 "" H 7500 2050 50  0001 C CNN
+F 2 "Diodes_SMD:D_SOD-123F" H 7500 2050 50  0001 C CNN
 F 3 "~" H 7500 2050 50  0001 C CNN
 	1    7500 2050
@@
 F 0 "D5" H 6050 5566 50  0000 C CNN
 F 1 "1N914" H 6050 5475 50  0000 C CNN
-F 2 "" H 6050 5350 50  0001 C CNN
+F 2 "Diodes_SMD:D_SOD-123F" H 6050 5350 50  0001 C CNN
 F 3 "~" H 6050 5350 50  0001 C CNN
 	1    6050 5350
@@
 F 0 "D4" H 7450 4216 50  0000 C CNN
 F 1 "1N914" H 7450 4125 50  0000 C CNN
-F 2 "" H 7450 4000 50  0001 C CNN
+F 2 "Diodes_SMD:D_SOD-123F" H 7450 4000 50  0001 C CNN
 F 3 "~" H 7450 4000 50  0001 C CNN
 	1    7450 4000
@@
 F 0 "D3" H 7450 3434 50  0000 C CNN
 F 1 "1N914" H 7450 3525 50  0000 C CNN
-F 2 "" H 7450 3650 50  0001 C CNN
+F 2 "Diodes_SMD:D_SOD-123F" H 7450 3650 50  0001 C CNN
 F 3 "~" H 7450 3650 50  0001 C CNN
 	1    7450 3650
@@
 Wire Wire Line
 	9900 3400 10050 3400
+Text Notes 7250 3600 0    50   ~ 0
+Attack Time\n
+Text Notes 7250 4150 0    50   ~ 0
+Release Time\n
 $EndSCHEMATC
