File: SLMMK1/CVPal.sch (KiCad schematic (older format))
At the start: 23 parts, among them J2 USB_B_Micro, J3 AVR-ISP-6, U8 ATtiny84-20PU, U9 MCP4822, Y1 Crystal

Commit message: Finished version
Parts:
- removed J2: USB_B_Micro, symbol Connector:USB_B_Micro
- added J2: USB_B, Connectors:USB_B, symbol Connector:USB_B
- C19, C23: value CP1 -> 100nF
- C20, C21: value CP1 -> 18pF
- C24: value CP1 -> 4.7uF
- D13: footprint (none) -> LEDs:LED_D5.0mm
- D14, D15: footprint (none) -> Diodes_SMD:D_SOD-123F
- L1: footprint (none) -> Inductors_THT:L_Axial_L9.5mm_D4.0mm_P5.08mm_Vertical_Fastron_SMCC
- R29: value R -> 0R
- R44, R48, R51, R53: value R -> 220R
Changed lines of the file:
@@
 $EndDescr
-$Comp
-L Connector:USB_B_Micro J2
-U 1 1 5BD74F3D
-P 4400 3550
-F 0 "J2" H 4455 4017 50  0000 C CNN
-F 1 "USB_B_Micro" H 4455 3926 50  0000 C CNN
-F 2 "" H 4550 3500 50  0001 C CNN
-F 3 "~" H 4550 3500 50  0001 C CNN
-	1    4400 3550
-	1    0    0    -1
-$EndComp
 $Comp
 L Device:Crystal Y1
@@
 P 5850 2150
 F 0 "C20" V 6102 2150 50  0000 C CNN
-F 1 "CP1" V 6011 2150 50  0000 C CNN
+F 1 "18pF" V 6011 2150 50  0000 C CNN
 F 2 "Capacitors_SMD:C_0805_HandSoldering" H 5850 2150 50  0001 C CNN
 F 3 "~" H 5850 2150 50  0001 C CNN
@@
 P 5850 2550
 F 0 "C21" V 6102 2550 50  0000 C CNN
-F 1 "CP1" V 6011 2550 50  0000 C CNN
+F 1 "18pF" V 6011 2550 50  0000 C CNN
 F 2 "Capacitors_SMD:C_0805_HandSoldering" H 5850 2550 50  0001 C CNN
 F 3 "~" H 5850 2550 50  0001 C CNN
@@
 	4400 4050 4400 3950
 Connection ~ 4350 4050
-NoConn ~ 4700 3750
 $Comp
 L Device:R R37
@@
 U 1 1 5BD7C9F2
 P 5150 2700
-F 0 "R29" V 5200 3000 50  0000 C CNN
-F 1 "R" V 5200 2900 50  0000 C CNN
+F 0 "R29" V 5250 2700 50  0000 C CNN
+F 1 "0R" V 5050 2750 50  0000 C CNN
 F 2 "Resistors_SMD:R_0805_HandSoldering" V 5080 2700 50  0001 C CNN
 F 3 "~" H 5150 2700 50  0001 C CNN
@@
 F 0 "D14" V 4754 3979 50  0000 L CNN
 F 1 "1N5227" V 4845 3979 50  0000 L CNN
-F 2 "" H 4800 3900 50  0001 C CNN
+F 2 "Diodes_SMD:D_SOD-123F" H 4800 3900 50  0001 C CNN
 F 3 "~" H 4800 3900 50  0001 C CNN
 	1    4800 3900
@@
 F 0 "D15" V 5204 3979 50  0000 L CNN
 F 1 "1N5227" V 5295 3979 50  0000 L CNN
-F 2 "" H 5250 3900 50  0001 C CNN
+F 2 "Diodes_SMD:D_SOD-123F" H 5250 3900 50  0001 C CNN
 F 3 "~" H 5250 3900 50  0001 C CNN
 	1    5250 3900
@@
 F 0 "L1" H 8109 954 50  0000 R CNN
 F 1 "L" H 8109 1045 50  0000 R CNN
-F 2 "" H 8150 1000 50  0001 C CNN
+F 2 "Inductors_THT:L_Axial_L9.5mm_D4.0mm_P5.08mm_Vertical_Fastron_SMCC" H 8150 1000 50  0001 C CNN
 F 3 "~" H 8150 1000 50  0001 C CNN
 	1    8150 1000
@@
 P 8000 1400
 F 0 "C23" H 8115 1446 50  0000 L CNN
-F 1 "CP1" H 8115 1355 50  0000 L CNN
+F 1 "100nF" H 8115 1355 50  0000 L CNN
 F 2 "Capacitors_SMD:C_0805_HandSoldering" H 8000 1400 50  0001 C CNN
 F 3 "~" H 8000 1400 50  0001 C CNN
@@
 P 8350 1400
 F 0 "C24" H 8465 1446 50  0000 L CNN
-F 1 "CP1" H 8465 1355 50  0000 L CNN
+F 1 "4.7uF" H 8465 1355 50  0000 L CNN
 F 2 "Capacitors_SMD:C_0805_HandSoldering" H 8350 1400 50  0001 C CNN
 F 3 "~" H 8350 1400 50  0001 C CNN
@@
 P 3400 1800
 F 0 "C19" H 3515 1846 50  0000 L CNN
-F 1 "CP1" H 3515 1755 50  0000 L CNN
+F 1 "100nF" H 3515 1755 50  0000 L CNN
 F 2 "Capacitors_SMD:C_0805_HandSoldering" H 3400 1800 50  0001 C CNN
 F 3 "~" H 3400 1800 50  0001 C CNN
@@
 P 8450 1900
 F 0 "R44" V 8243 1900 50  0000 C CNN
-F 1 "R" V 8334 1900 50  0000 C CNN
+F 1 "220R" V 8334 1900 50  0000 C CNN
 F 2 "Resistors_SMD:R_0805_HandSoldering" V 8380 1900 50  0001 C CNN
 F 3 "~" H 8450 1900 50  0001 C CNN
@@
 P 8450 2200
 F 0 "R48" V 8243 2200 50  0000 C CNN
-F 1 "R" V 8334 2200 50  0000 C CNN
+F 1 "220R" V 8334 2200 50  0000 C CNN
 F 2 "Resistors_SMD:R_0805_HandSoldering" V 8380 2200 50  0001 C CNN
 F 3 "~" H 8450 2200 50  0001 C CNN
@@
 P 8500 2500
 F 0 "R51" V 8293 2500 50  0000 C CNN
-F 1 "R" V 8384 2500 50  0000 C CNN
+F 1 "220R" V 8384 2500 50  0000 C CNN
 F 2 "Resistors_SMD:R_0805_HandSoldering" V 8430 2500 50  0001 C CNN
 F 3 "~" H 8500 2500 50  0001 C CNN
@@
 P 8500 2800
 F 0 "R53" V 8293 2800 50  0000 C CNN
-F 1 "R" V 8384 2800 50  0000 C CNN
+F 1 "220R" V 8384 2800 50  0000 C CNN
 F 2 "Resistors_SMD:R_0805_HandSoldering" V 8430 2800 50  0001 C CNN
 F 3 "~" H 8500 2800 50  0001 C CNN
@@
 F 0 "D13" V 3238 3883 50  0000 R CNN
 F 1 "LED" V 3147 3883 50  0000 R CNN
-F 2 "" H 3200 4000 50  0001 C CNN
+F 2 "LEDs:LED_D5.0mm" H 3200 4000 50  0001 C CNN
 F 3 "~" H 3200 4000 50  0001 C CNN
 	1    3200 4000
@@
 	1    0    0    -1
 $EndComp
+$Comp
+L Connector:USB_B J2
+U 1 1 5BC0F38B
+P 4400 3550
+F 0 "J2" H 4455 4017 50  0000 C CNN
+F 1 "USB_B" H 4455 3926 50  0000 C CNN
+F 2 "Connectors:USB_B" H 4550 3500 50  0001 C CNN
+F 3 " ~" H 4550 3500 50  0001 C CNN
+	1    4400 3550
+	1    0    0    -1
+$EndComp
+NoConn ~ 4700 3750
 $EndSCHEMATC
