File: SLMMK1/SLMMK1.sch (KiCad schematic (older format))
At the start: 15 parts, among them J1 AudioJack2_Ground, J4 AudioJack2_Ground, J5 AudioJack2_Ground, J6 AudioJack2_Ground, J7 AudioJack2_Ground, J8 AudioJack2_Ground, J9 Screw_Terminal_01x03, SW19 SW_DPST, SW20 SW_SPDT, SW21 SW_SPDT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

Commit message: Finished version
Parts:
- J1, J4, J5, J8: footprint (none) -> TomsLib:AudioJack_Out
- J6, J7: footprint (none) -> TomsLib:1340604
Connections:
- net labels added: +9Vin, -9Vin
- wire segments 107 -> 110
Changed lines of the file:
@@
 	5500 1800 5900 1800
 Wire Wire Line
-	5900 1950 5900 1800
+	5900 1950 5900 1900
 Connection ~ 5900 1800
-Wire Wire Line
-	5900 1100 5900 850
 Connection ~ 5900 1100
 Wire Wire Line
 	5900 1400 5900 1450
-Wire Wire Line
-	6150 1450 5900 1450
 Connection ~ 5900 1450
 Wire Wire Line
@@
 F 0 "J1" H 8817 3679 50  0000 R CNN
 F 1 "AudioJack2_Ground" H 8817 3770 50  0000 R CNN
-F 2 "" H 9050 3700 50  0001 C CNN
+F 2 "TomsLib:AudioJack_Out" H 9050 3700 50  0001 C CNN
 F 3 "~" H 9050 3700 50  0001 C CNN
 	1    9050 3700
@@
 F 0 "J4" H 1317 2229 50  0000 R CNN
 F 1 "AudioJack2_Ground" H 1317 2320 50  0000 R CNN
-F 2 "" H 1550 2250 50  0001 C CNN
+F 2 "TomsLib:AudioJack_Out" H 1550 2250 50  0001 C CNN
 F 3 "~" H 1550 2250 50  0001 C CNN
 	1    1550 2250
@@
 F 0 "J5" H 1317 2629 50  0000 R CNN
 F 1 "AudioJack2_Ground" H 1317 2720 50  0000 R CNN
-F 2 "" H 1550 2650 50  0001 C CNN
+F 2 "TomsLib:AudioJack_Out" H 1550 2650 50  0001 C CNN
 F 3 "~" H 1550 2650 50  0001 C CNN
 	1    1550 2650
@@
 F 0 "J6" H 2217 3879 50  0000 R CNN
 F 1 "AudioJack2_Ground" H 2217 3970 50  0000 R CNN
-F 2 "" H 2450 3900 50  0001 C CNN
+F 2 "TomsLib:1340604" H 2450 3900 50  0001 C CNN
 F 3 "~" H 2450 3900 50  0001 C CNN
 	1    2450 3900
@@
 F 0 "J7" H 2217 4229 50  0000 R CNN
 F 1 "AudioJack2_Ground" H 2217 4320 50  0000 R CNN
-F 2 "" H 2450 4250 50  0001 C CNN
+F 2 "TomsLib:1340604" H 2450 4250 50  0001 C CNN
 F 3 "~" H 2450 4250 50  0001 C CNN
 	1    2450 4250
@@
 F 0 "J8" H 1317 1779 50  0000 R CNN
 F 1 "AudioJack2_Ground" H 1317 1870 50  0000 R CNN
-F 2 "" H 1550 1800 50  0001 C CNN
+F 2 "TomsLib:AudioJack_Out" H 1550 1800 50  0001 C CNN
 F 3 "~" H 1550 1800 50  0001 C CNN
 	1    1550 1800
@@
 	1    0    0    -1
 $EndComp
+$Comp
+L power:PWR_FLAG #FLG0102
+U 1 1 5BBFD906
+P 5900 1900
+F 0 "#FLG0102" H 5900 1975 50  0001 C CNN
+F 1 "PWR_FLAG" V 5900 2028 50  0000 L CNN
+F 2 "" H 5900 1900 50  0001 C CNN
+F 3 "~" H 5900 1900 50  0001 C CNN
+	1    5900 1900
+	0    1    1    0
+$EndComp
+Connection ~ 5900 1900
+Wire Wire Line
+	5900 1900 5900 1800
+Wire Wire Line
+	5900 850  5900 950
+Wire Wire Line
+	5900 1450 6150 1450
+$Comp
+L power:PWR_FLAG #FLG0101
+U 1 1 5BC090A0
+P 6150 950
+F 0 "#FLG0101" H 6150 1025 50  0001 C CNN
+F 1 "PWR_FLAG" H 6150 1124 50  0000 C CNN
+F 2 "" H 6150 950 50  0001 C CNN
+F 3 "~" H 6150 950 50  0001 C CNN
+	1    6150 950
+	1    0    0    -1
+$EndComp
+Wire Wire Line
+	6150 950  5900 950
+Connection ~ 5900 950
+Wire Wire Line
+	5900 950  5900 1100
+Text Label 4600 1100 0    50   ~ 0
++9Vin
+Text Label 4500 1800 0    50   ~ 0
+-9Vin
 $EndSCHEMATC
