File: SLMMK1/LFO.sch (KiCad schematic (older format))
At the start: 19 parts, among them Q9 2N3904, SW16 SW_SPDT_MSM, SW17 SW_SPST, SW18 SW_SPDT, U7 TL074

Commit message: Finished version
Parts:
- D10, D9: footprint (none) -> Diodes_SMD:D_SOD-123F
- D6: footprint (none) -> LEDs:LED_D5.0mm
- Q9: footprint Package_TO_SOT_THT:TO-92_Inline -> TO_SOT_Packages_THT:TO-92_Inline_Wide
Other:
- note added: "Frequency\n"
- note added: "Level\n"
Changed lines of the file:
@@
 F 0 "D10" H 4450 4166 50  0000 C CNN
 F 1 "1N914" H 4450 4075 50  0000 C CNN
-F 2 "" H 4450 3950 50  0001 C CNN
+F 2 "Diodes_SMD:D_SOD-123F" H 4450 3950 50  0001 C CNN
 F 3 "~" H 4450 3950 50  0001 C CNN
 	1    4450 3950
@@
 F 0 "D9" H 4450 3434 50  0000 C CNN
 F 1 "1N914" H 4450 3525 50  0000 C CNN
-F 2 "" H 4450 3650 50  0001 C CNN
+F 2 "Diodes_SMD:D_SOD-123F" H 4450 3650 50  0001 C CNN
 F 3 "~" H 4450 3650 50  0001 C CNN
 	1    4450 3650
@@
 F 0 "Q9" H 7041 5796 50  0000 L CNN
 F 1 "2N3904" H 7041 5705 50  0000 L CNN
-F 2 "Package_TO_SOT_THT:TO-92_Inline" H 7050 5675 50  0001 L CIN
+F 2 "TO_SOT_Packages_THT:TO-92_Inline_Wide" H 7050 5675 50  0001 L CIN
 F 3 "https://www.fairchildsemi.com/datasheets/2N/2N3904.pdf" H 6850 5750 50  0001 L CNN
 	1    6850 5750
@@
 F 0 "D6" V 6988 5983 50  0000 R CNN
 F 1 "LED" V 6897 5983 50  0000 R CNN
-F 2 "" H 6950 6100 50  0001 C CNN
+F 2 "LEDs:LED_D5.0mm" H 6950 6100 50  0001 C CNN
 F 3 "~" H 6950 6100 50  0001 C CNN
 	1    6950 6100
@@
 Wire Wire Line
 	6500 4350 6650 4350
+Text Notes 4350 4350 0    50   ~ 0
+Frequency\n
+Text Notes 9000 3700 0    50   ~ 0
+Level\n
 $EndSCHEMATC

Commit message: Fixed obvious bugs in schematics, pcb/gerbers not updated
Changed lines of the file:
@@
 F 3 "http://www.ti.com/lit/ds/symlink/tl071.pdf" H 6050 4550 50  0001 C CNN
 	1    6000 4350
-	1    0    0    -1
+	1    0    0    1
 $EndComp
 $Comp
@@
 F 3 "http://www.ti.com/lit/ds/symlink/tl071.pdf" H 7700 4450 50  0001 C CNN
 	2    7650 4250
-	1    0    0    -1
+	1    0    0    1
 $EndComp
 $Comp
