File: SLMMK1/NoiseGen.sch (KiCad schematic (older format))
At the start: 12 parts, among them Q7 2N3904, U7 TL074

Commit message: Finished version
Parts:
- Q7: footprint Package_TO_SOT_THT:TO-92_Inline -> TO_SOT_Packages_THT:TO-92_Inline_Wide
Changed lines of the file:
@@
 F 0 "Q7" H 5291 3996 50  0000 L CNN
 F 1 "2N3904" H 5291 3905 50  0000 L CNN
-F 2 "Package_TO_SOT_THT:TO-92_Inline" H 5300 3875 50  0001 L CIN
+F 2 "TO_SOT_Packages_THT:TO-92_Inline_Wide" H 5300 3875 50  0001 L CIN
 F 3 "https://www.fairchildsemi.com/datasheets/2N/2N3904.pdf" H 5100 3950 50  0001 L CNN
 	1    5100 3950

Commit message: Fixed obvious bugs in schematics, pcb/gerbers not updated
Connections:
- wire segments 41 -> 37
