File: SLMMK1/VCA.sch (KiCad schematic (older format))
At the start: 17 parts, among them SW4 SW_SPST, SW5 SW_SPST, SW6 SW_SPDT, U3 LM13700

Commit message: Finished version
Parts:
- RV19: value R_POT -> 100K
Changed lines of the file:
@@
 P 2350 2050
 F 0 "RV19" H 2280 2096 50  0000 R CNN
-F 1 "R_POT" H 2280 2005 50  0000 R CNN
+F 1 "100K" H 2280 2005 50  0000 R CNN
 F 2 "Pin_Headers:Pin_Header_Straight_1x03_Pitch2.54mm" H 2350 2050 50  0001 C CNN
 F 3 "~" H 2350 2050 50  0001 C CNN

Commit message: Fixed obvious bugs in schematics, pcb/gerbers not updated
Parts:
- R26: value 100K -> 10K
Changed lines of the file:
@@
 $Descr A4 11693 8268
 encoding utf-8
-Sheet 6 9
+Sheet 5 9
 Title ""
 Date ""
@@
 P 4550 3450
 F 0 "R26" H 4480 3404 50  0000 R CNN
-F 1 "100K" H 4480 3495 50  0000 R CNN
+F 1 "10K" H 4480 3495 50  0000 R CNN
 F 2 "Resistors_SMD:R_0805_HandSoldering" V 4480 3450 50  0001 C CNN
 F 3 "~" H 4550 3450 50  0001 C CNN
