File: SLMMK1/VCF.sch (KiCad schematic (older format))
At the start: 25 parts, among them SW7 SW_SPST, SW8 SW_SPST, U4 LM13700

Commit message: Fixed obvious bugs in schematics, pcb/gerbers not updated
Parts:
- added C4: 560pF, Capacitors_SMD:C_0805_HandSoldering, symbol Device:CP1
- added R43: 20K, Resistors_SMD:R_0805_HandSoldering, symbol Device:R
Changed lines of the file:
@@
 Wire Wire Line
 	4750 4000 4850 4000
-Wire Wire Line
-	4850 4050 4850 4000
 Connection ~ 4850 4000
 Wire Wire Line
@@
 $EndComp
 NoConn ~ 6400 4200
+$Comp
+L Device:CP1 C4
+U 1 1 5BE41C46
+P 4850 4250
+F 0 "C4" H 4965 4296 50  0000 L CNN
+F 1 "560pF" H 4965 4205 50  0000 L CNN
+F 2 "Capacitors_SMD:C_0805_HandSoldering" H 4850 4250 50  0001 C CNN
+F 3 "~" H 4850 4250 50  0001 C CNN
+	1    4850 4250
+	1    0    0    -1
+$EndComp
+$Comp
+L power:GND #PWR0177
+U 1 1 5BE41CEC
+P 4850 4400
+F 0 "#PWR0177" H 4850 4150 50  0001 C CNN
+F 1 "GND" H 4855 4227 50  0000 C CNN
+F 2 "" H 4850 4400 50  0001 C CNN
+F 3 "" H 4850 4400 50  0001 C CNN
+	1    4850 4400
+	1    0    0    -1
+$EndComp
+Wire Wire Line
+	4850 4000 4850 4100
+$Comp
+L Device:R R43
+U 1 1 5BE43AE5
+P 7700 5100
+F 0 "R43" H 7630 5054 50  0000 R CNN
+F 1 "20K" H 7630 5145 50  0000 R CNN
+F 2 "Resistors_SMD:R_0805_HandSoldering" V 7630 5100 50  0001 C CNN
+F 3 "~" H 7700 5100 50  0001 C CNN
+	1    7700 5100
+	-1   0    0    1
+$EndComp
+$Comp
+L power:-9V #PWR?
+U 1 1 5BE43B5D
+P 7700 5250
+F 0 "#PWR?" H 7700 5125 50  0001 C CNN
+F 1 "-9V" H 7715 5423 50  0000 C CNN
+F 2 "" H 7700 5250 50  0001 C CNN
+F 3 "" H 7700 5250 50  0001 C CNN
+	1    7700 5250
+	-1   0    0    1
+$EndComp
+Connection ~ 7700 4950
 $EndSCHEMATC
