File: SLMMK1/VCO1.sch (KiCad schematic (older format))
At the start: 30 parts, among them Q1 2N3904, Q3 2N3904, Q5 Q_NJFET_DGS, SW11 SW_SPST, SW13 SW_SPST, U5 TL074

Commit message: Finished version
Parts:
- removed Q5: Q_NJFET_DGS, symbol Device:Q_NJFET_DGS
- added Q5: Q_NJFET_DSG, TO_SOT_Packages_THT:TO-92_Inline_Wide, symbol Device:Q_NJFET_DSG
- Q1, Q3: footprint Package_TO_SOT_THT:TO-92_Inline -> TO_SOT_Packages_THT:TO-92_Inline_Wide
Changed lines of the file:
@@
 F 0 "Q3" H 5941 3854 50  0000 L CNN
 F 1 "2N3904" H 5941 3945 50  0000 L CNN
-F 2 "Package_TO_SOT_THT:TO-92_Inline" H 5950 3825 50  0001 L CIN
+F 2 "TO_SOT_Packages_THT:TO-92_Inline_Wide" H 5950 3825 50  0001 L CIN
 F 3 "https://www.fairchildsemi.com/datasheets/2N/2N3904.pdf" H 5750 3900 50  0001 L CNN
 	1    5750 3900
@@
 F 0 "Q1" H 5941 3346 50  0000 L CNN
 F 1 "2N3904" H 5941 3255 50  0000 L CNN
-F 2 "Package_TO_SOT_THT:TO-92_Inline" H 5950 3225 50  0001 L CIN
+F 2 "TO_SOT_Packages_THT:TO-92_Inline_Wide" H 5950 3225 50  0001 L CIN
 F 3 "https://www.fairchildsemi.com/datasheets/2N/2N3904.pdf" H 5750 3300 50  0001 L CNN
 	1    5750 3300
@@
 Connection ~ 6300 2650
 $Comp
-L Device:Q_NJFET_DGS Q5
-U 1 1 5BC59363
-P 6300 4450
-F 0 "Q5" V 6300 4150 50  0000 C CNN
-F 1 "Q_NJFET_DGS" V 6200 4050 50  0000 C CNN
-F 2 "" H 6500 4550 50  0001 C CNN
-F 3 "~" H 6300 4450 50  0001 C CNN
-	1    6300 4450
-	0    -1   1    0
-$EndComp
-$Comp
 L Device:CP1 C8
 U 1 1 5BC5B376
@@
 Wire Wire Line
 	2050 2100 2050 2050
+$Comp
+L Device:Q_NJFET_DSG Q5
+U 1 1 5BBF95C4
+P 6300 4450
+F 0 "Q5" V 6536 4450 50  0000 C CNN
+F 1 "Q_NJFET_DSG" V 6627 4450 50  0000 C CNN
+F 2 "TO_SOT_Packages_THT:TO-92_Inline_Wide" H 6500 4550 50  0001 C CNN
+F 3 "~" H 6300 4450 50  0001 C CNN
+	1    6300 4450
+	0    1    1    0
+$EndComp
 $EndSCHEMATC

Commit message: Fixed obvious bugs in schematics, pcb/gerbers not updated
Connections:
- wire segments 100 -> 99
Changed lines of the file:
@@
 $EndComp
 Wire Wire Line
-	5850 6150 5850 5350
+	5850 5400 5850 5350
 Wire Wire Line
 	5850 5350 6000 5350
@@
 $EndComp
 Wire Wire Line
-	6500 6150 5850 6150
-Wire Wire Line
 	6500 6450 6800 6450
-Connection ~ 6500 6150
 Wire Wire Line
 	6500 6150 6900 6150
@@
 	0    1    1    0
 $EndComp
+$Comp
+L power:GND #PWR0178
+U 1 1 5BE1C55D
+P 5850 5400
+F 0 "#PWR0178" H 5850 5150 50  0001 C CNN
+F 1 "GND" H 5855 5227 50  0000 C CNN
+F 2 "" H 5850 5400 50  0001 C CNN
+F 3 "" H 5850 5400 50  0001 C CNN
+	1    5850 5400
+	1    0    0    -1
+$EndComp
 $EndSCHEMATC
