File: SLMMK1/VCO2.sch (KiCad schematic (older format))
At the start: 44 parts, among them Q2 2N3904, Q4 2N3904, Q6 Q_NJFET_DGS, SW10 SW_SPDT, SW12 SW_SPST, SW14 SW_SPST, SW15 SW_SPST, U2 TL072, U6 TL074

Commit message: Finished version
Parts:
- removed Q6: Q_NJFET_DGS, symbol Device:Q_NJFET_DGS
- added Q6: Q_NJFET_DSG, TO_SOT_Packages_THT:TO-92_Inline_Wide, symbol Device:Q_NJFET_DSG
- D11, D12: footprint (none) -> Diodes_SMD:D_SOD-123F
- Q2, Q4: footprint Package_TO_SOT_THT:TO-92_Inline -> TO_SOT_Packages_THT:TO-92_Inline_Wide
Other:
- note added: "Coarse\n"
- note added: "Fine\n"
Changed lines of the file:
@@
 F 0 "Q4" H 5741 3554 50  0000 L CNN
 F 1 "2N3904" H 5741 3645 50  0000 L CNN
-F 2 "Package_TO_SOT_THT:TO-92_Inline" H 5750 3525 50  0001 L CIN
+F 2 "TO_SOT_Packages_THT:TO-92_Inline_Wide" H 5750 3525 50  0001 L CIN
 F 3 "https://www.fairchildsemi.com/datasheets/2N/2N3904.pdf" H 5550 3600 50  0001 L CNN
 	1    5550 3600
@@
 F 0 "Q2" H 5741 3046 50  0000 L CNN
 F 1 "2N3904" H 5741 2955 50  0000 L CNN
-F 2 "Package_TO_SOT_THT:TO-92_Inline" H 5750 2925 50  0001 L CIN
+F 2 "TO_SOT_Packages_THT:TO-92_Inline_Wide" H 5750 2925 50  0001 L CIN
 F 3 "https://www.fairchildsemi.com/datasheets/2N/2N3904.pdf" H 5550 3000 50  0001 L CNN
 	1    5550 3000
@@
 Connection ~ 6100 2350
 $Comp
-L Device:Q_NJFET_DGS Q?
-U 1 1 5BCAE57A
-P 6100 4150
-AR Path="/5BB9042D/5BCAE57A" Ref="Q?"  Part="1"
-AR Path="/5BCAB8D3/5BCAE57A" Ref="Q6"  Part="1"
-F 0 "Q6" V 6100 3850 50  0000 C CNN
-F 1 "Q_NJFET_DGS" V 6000 3750 50  0000 C CNN
-F 2 "" H 6300 4250 50  0001 C CNN
-F 3 "~" H 6100 4150 50  0001 C CNN
-	1    6100 4150
-	0    -1   1    0
-$EndComp
-$Comp
 L Device:CP1 C?
 U 1 1 5BCAE581
@@
 F 0 "D12" H 8050 4834 50  0000 C CNN
 F 1 "1N914" H 8050 4925 50  0000 C CNN
-F 2 "" H 8050 5050 50  0001 C CNN
+F 2 "Diodes_SMD:D_SOD-123F" H 8050 5050 50  0001 C CNN
 F 3 "~" H 8050 5050 50  0001 C CNN
 	1    8050 5050
@@
 F 0 "D11" H 8050 5384 50  0000 C CNN
 F 1 "1N914" H 8050 5475 50  0000 C CNN
-F 2 "" H 8050 5600 50  0001 C CNN
+F 2 "Diodes_SMD:D_SOD-123F" H 8050 5600 50  0001 C CNN
 F 3 "~" H 8050 5600 50  0001 C CNN
 	1    8050 5600
@@
 Text Notes 7350 2400 0    50   ~ 0
 Pulse Width
+$Comp
+L Device:Q_NJFET_DSG Q6
+U 1 1 5BBF9910
+P 6100 4150
+F 0 "Q6" V 6336 4150 50  0000 C CNN
+F 1 "Q_NJFET_DSG" V 6427 4150 50  0000 C CNN
+F 2 "TO_SOT_Packages_THT:TO-92_Inline_Wide" H 6300 4250 50  0001 C CNN
+F 3 "~" H 6100 4150 50  0001 C CNN
+	1    6100 4150
+	0    1    1    0
+$EndComp
+Text Notes 2850 2300 0    50   ~ 0
+Fine\n
+Text Notes 3150 1700 0    50   ~ 0
+Coarse\n
 $EndSCHEMATC

Commit message: Fixed obvious bugs in schematics, pcb/gerbers not updated
Connections:
- wire segments 124 -> 123
Changed lines of the file:
@@
 $EndComp
-Wire Wire Line
-	5650 5850 5650 5050
 Wire Wire Line
 	5650 5050 5800 5050
@@
 $EndComp
 Wire Wire Line
-	6300 5850 5650 5850
-Wire Wire Line
 	6300 6150 6600 6150
-Connection ~ 6300 5850
 Wire Wire Line
 	6300 5850 6700 5850
@@
 Text Notes 3150 1700 0    50   ~ 0
 Coarse\n
+$Comp
+L power:GND #PWR?
+U 1 1 5BE2936D
+P 5650 5100
+AR Path="/5BB9042D/5BE2936D" Ref="#PWR?"  Part="1"
+AR Path="/5BCAB8D3/5BE2936D" Ref="#PWR0179"  Part="1"
+F 0 "#PWR0179" H 5650 4850 50  0001 C CNN
+F 1 "GND" H 5655 4927 50  0000 C CNN
+F 2 "" H 5650 5100 50  0001 C CNN
+F 3 "" H 5650 5100 50  0001 C CNN
+	1    5650 5100
+	1    0    0    -1
+$EndComp
+Wire Wire Line
+	5650 5050 5650 5100
 $EndSCHEMATC
